File: schematic/main/main.kicad_pcb (KiCad board)
At the start: 2 copper layers, 0 parts

Commit message: PCBs started!
Parts:
- added A1: Arduino_Pro_Mini, arduino_pro_mini:arduino_pro_mini, F.Cu at (134.6, 109.2)
- added A2: Teensy_32, teensy_32:teensy_32, F.Cu at (129.5, 53.3)
- added C1: 1000u, Capacitors_THT:CP_Radial_D12.5mm_P5.00mm, F.Cu at (131.1, 98.4)
- added CON1: Left Pumps, Pin_Headers:Pin_Header_Angled_1x15_Pitch2.54mm, F.Cu at (149.9, 53.3)
- added CON2: Right Pumps, Pin_Headers:Pin_Header_Angled_1x15_Pitch2.54mm, F.Cu at (124.5, 88.9)
- added J1: Button, Pin_Headers:Pin_Header_Straight_1x02_Pitch2.54mm, F.Cu at (131.0, 117.8)
- added J2: Sensor, Pin_Headers:Pin_Header_Straight_1x03_Pitch2.54mm, F.Cu at (131.0, 122.1)
- added J3: 5V Relay, Pin_Headers:Pin_Header_Straight_1x03_Pitch2.54mm, F.Cu at (144.5, 141.2)
- added J4: 24V Relay, Pin_Headers:Pin_Header_Straight_1x03_Pitch2.54mm, F.Cu at (134.9, 141.2)
- added J5: LEDs, Pin_Headers:Pin_Header_Straight_1x03_Pitch2.54mm, F.Cu at (131.0, 109.1)
- added J6: Fan, Pin_Headers:Pin_Header_Straight_1x02_Pitch2.54mm, F.Cu at (218.4, 144.8)
- added JP1: PRG, Pin_Headers:Pin_Header_Straight_1x02_Pitch2.54mm, F.Cu at (144.8, 48.3)
- added M1: LLC4, logic_level_converter:LLC4, F.Cu at (149.9, 93.0)
- added R1: 330, Resistors_THT:R_Axial_DIN0309_L9.0mm_D3.2mm_P2.54mm_Vertical, F.Cu at (129.6, 113.3)
- added T1: 5V, Wire_Pads:SolderWirePad_2x_1-5mmDrill, F.Cu at (177.8, 132.1)
- added T2: 5VS, Wire_Pads:SolderWirePad_2x_1-5mmDrill, F.Cu at (223.1, 120.2)
- added T3: 24VS, Wire_Pads:SolderWirePad_2x_1-5mmDrill, F.Cu at (127.0, 48.0)
- added T4: GND, Wire_Pads:SolderWirePad_2x_1-5mmDrill, F.Cu at (252.3, 110.2)
Routing:
- net /3.3V: track 0.00 -> 68.6 mm, vias 0 -> 2
- net /5VS: track 0.00 -> 57.4 mm, vias 0 -> 2
- net /~ENABLE: track 0.00 -> 45.7 mm, vias 0 -> 2
- net /DIR: track 0.00 -> 41.6 mm
- net /A2_D1: track 0.00 -> 28.6 mm, vias 0 -> 2
- net /A2_D0: track 0.00 -> 18.8 mm, vias 0 -> 2
- net /P7: track 0.00 -> 7.18 mm
- net /P6: track 0.00 -> 7.18 mm
- net /P5: track 0.00 -> 7.18 mm
- net /P4: track 0.00 -> 7.18 mm
- net /P9: track 0.00 -> 7.18 mm
- net /P8: track 0.00 -> 7.18 mm
- net /P11: track 0.00 -> 7.18 mm
- net /P10: track 0.00 -> 7.18 mm
- net /5VS_2: track 0.00 -> 6.64 mm
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Other:
- net class 24V Power added: clearance 0.1524, trace_width 0.508, via_dia 0.6858, via_drill 0.3302
- net class Default: trace_width 0.1524 -> 0.2032
- net class Power: trace_width 0.4572 -> 0.3048

Commit message: Finished board designs.
Parts:
- removed the CON1 at (149.9, 53.3)
- added CON2: Right, Pin_Headers:Pin_Header_Angled_1x15_Pitch2.54mm, F.Cu at (124.5, 88.9)
- added J7: Pi, Pin_Headers:Pin_Header_Straight_1x02_Pitch2.54mm, F.Cu at (130.6, 109.2)
- added REF**: MountingHole_3mm, Mounting_Holes:MountingHole_3mm, F.Cu at (123.8, 47.4)
- added REF**: MountingHole_3mm, Mounting_Holes:MountingHole_3mm, F.Cu at (150.5, 47.4)
- added REF**: MountingHole_3mm, Mounting_Holes:MountingHole_3mm, F.Cu at (123.8, 142.6)
- added REF**: MountingHole_3mm, Mounting_Holes:MountingHole_3mm, F.Cu at (150.5, 142.6)
- CON1: renamed from CON2; value Right Pumps -> Left
- R1: footprint Resistors_THT:R_Axial_DIN0309_L9.0mm_D3.2mm_P2.54mm_Vertical -> Resistors_THT:R_Axial_DIN0207_L6.3mm_D2.5mm_P2.54mm_Vertical
- T1, T2, T3, T4: footprint Wire_Pads:SolderWirePad_2x_1-5mmDrill -> spade_terminal:Spade_Terminal_1_4
- moved T4 130.6 mm to (123.1, 129.3), turned to 270 degrees
- moved T2 100.8 mm to (123.1, 107.5), turned to 90 degrees
- moved J6 88.2 mm to (130.6, 137.2), turned to 90 degrees
- moved T1 56.4 mm to (123.1, 118.4), turned to 270 degrees
- moved T3 48.7 mm to (123.1, 96.5), turned to 90 degrees
- moved CON1 43.7 mm to (149.8, 53.3), turned to 0 degrees
- moved J1 14.3 mm to (130.6, 132.1), turned to 90 degrees
- moved M1 8.72 mm to (141.1, 92.7), turned to 0 degrees
- moved R1 6.39 mm to (131.6, 119.4), turned to 0 degrees
- moved J5 6.08 mm to (128.0, 114.4), turned to 90 degrees
- moved J2 5.74 mm to (128.0, 127.0), turned to 90 degrees
- moved J4 5.60 mm to (129.3, 141.8)
- moved J3 5.04 mm to (139.5, 141.8)
- moved C1 3.62 mm to (132.6, 95.1), turned to 270 degrees
- moved JP1 2.55 mm to (142.2, 48.0)
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Connections:
- A1 pad 5: /D2 -> /D2_2
- CON1 pad 10: /P12 -> /P4
- CON1 pad 11: /P13 -> /P5
- CON1 pad 12: /P14 -> /P6
- CON1 pad 13: /P15 -> /P7
- CON1 pad 3: /P8 -> /P0
- CON1 pad 4: /P9 -> /P1
- CON1 pad 5: /P10 -> /P2
- CON1 pad 6: /P11 -> /P3
- J1 pad 1: /D2 -> /GND
- J1 pad 2: /GND -> /D4
- J2 pad 1: /D3 -> /GND
- J2 pad 3: /GND -> /D3
- J3 pad 1: /5V -> /GND
- J3 pad 2: /D4 -> /D5
- J3 pad 3: /GND -> /5V
- J4 pad 1: /5V -> /GND
- J4 pad 2: /D5 -> /D6
- J4 pad 3: /GND -> /5V
- J5 pad 1: /5VS -> /GND
- J5 pad 2: Net-(J5-Pad2) -> /D2
- J5 pad 3: /GND -> /5VS
- J6 pad 1: /24VS -> /GND
- J6 pad 2: /GND -> /5VS
- M1 pad 1: (no net) -> /A2_D0
- M1 pad 11: (no net) -> /A1_D0
- M1 pad 12: (no net) -> /A1_D1
- M1 pad 2: (no net) -> /A2_D1
- M1 pad 5: /A2_D0 -> (no net)
- M1 pad 6: /A2_D1 -> (no net)
- M1 pad 7: /A1_D0 -> (no net)
- M1 pad 8: /A1_D1 -> (no net)
- R1 pad 1: /D6 -> /D2
- R1 pad 2: Net-(J5-Pad2) -> /D2_2
Routing:
- net /24VS: track 0.00 -> 111.8 mm
- net /5VS: track 57.4 -> 154.5 mm, vias 2 -> 6
- net /5V: track 0.00 -> 72.5 mm
- net /A1_D0: track 0.00 -> 31.0 mm
- net /A1_D1: track 0.00 -> 30.0 mm
- net /A2_D0: track 18.8 -> 42.6 mm
- net /D5: track 0.00 -> 17.3 mm
- net /D6: track 0.00 -> 14.3 mm
- net /GND: track 0.00 -> 13.3 mm
- net /A2_D1: track 28.6 -> 41.6 mm
- net /D4: track 0.00 -> 9.51 mm
- net /D3: track 0.00 -> 6.60 mm
- net /3.3V: track 68.6 -> 75.0 mm, vias 2 -> 3
- net /D2: track 0.00 -> 5.40 mm
- net /D2_2: track 0.00 -> 2.83 mm
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- added copper zone on B.Cu, net /GND
- added copper zone on F.Cu, net /GND
Other:
- board outline added: 33.5 x 102.1 mm
- net class 24V Power removed
- net class High Current added: clearance 0.1524, trace_width 2.54, via_dia 0.6858, via_drill 0.3302
- board text added: "Barbot Controller v1.0"

Commit message: Tweaked schematic and board
Parts:
- added J10: 5VS, Pin_Headers:Pin_Header_Straight_1x02_Pitch2.54mm, F.Cu at (134.6, 92.7)
- added J11: 5VS, Pin_Headers:Pin_Header_Straight_1x02_Pitch2.54mm, F.Cu at (137.9, 92.7)
- added J12: 5V, Pin_Headers:Pin_Header_Straight_1x02_Pitch2.54mm, F.Cu at (137.2, 143.5)
- added J13: 5V, Pin_Headers:Pin_Header_Straight_1x02_Pitch2.54mm, F.Cu at (140.5, 143.5)
- added J14: 5V, Pin_Headers:Pin_Header_Straight_1x02_Pitch2.54mm, F.Cu at (143.8, 143.5)
- added J15: 24S, Pin_Headers:Pin_Header_Straight_1x02_Pitch2.54mm, F.Cu at (129.5, 48.0)
- added J16: 3.3V, Pin_Headers:Pin_Header_Straight_1x02_Pitch2.54mm, F.Cu at (144.8, 89.7)
- added J8: 5VS, Pin_Headers:Pin_Header_Straight_1x02_Pitch2.54mm, F.Cu at (128.0, 92.7)
- added J9: 5VS, Pin_Headers:Pin_Header_Straight_1x02_Pitch2.54mm, F.Cu at (131.3, 92.7)
- C1: footprint Capacitors_THT:CP_Radial_D12.5mm_P5.00mm -> Capacitors_THT:CP_Radial_D10.0mm_P5.00mm
- J1: value Button -> LEDs; footprint Pin_Headers:Pin_Header_Straight_1x02_Pitch2.54mm -> Pin_Headers:Pin_Header_Straight_1x03_Pitch2.54mm
- J2: value Sensor -> Sensor0
- J3: value 5V Relay -> Sensor1
- J4: value 24V Relay -> Relay0
- J5: value LEDs -> Relay1
- J6: value Fan -> Relay2; footprint Pin_Headers:Pin_Header_Straight_1x02_Pitch2.54mm -> Pin_Headers:Pin_Header_Straight_1x03_Pitch2.54mm
- J7: value Pi -> Button
- moved C1 39.3 mm to (130.0, 134.4)
- moved J1 31.3 mm to (130.6, 100.8)
- moved J3 30.8 mm to (127.8, 113.3)
- moved J4 24.5 mm to (127.8, 117.3)
- moved J7 20.3 mm to (130.3, 129.5)
- moved J2 17.8 mm to (127.8, 109.2)
- moved R1 13.6 mm to (134.9, 106.2)
- moved J6 12.1 mm to (127.8, 125.5)
- moved J5 7.02 mm to (127.8, 121.4)
Connections:
- A1 pad 10: (no net) -> /D7
- A1 pad 11: (no net) -> /D8
- C1 pad 1: /5VS -> /5V
- J1 pad 2: /D4 -> /D2
- J3 pad 2: /D5 -> /5VS
- J3 pad 3: /5V -> /D4
- J4 pad 2: /D6 -> /D5
- J5 pad 2: /D2 -> /D6
- J5 pad 3: /5VS -> /5V
- J6 pad 2: /5VS -> /D7
- J7 pad 2: /5VS -> /D8
Routing:
- net /5VS: track 154.5 -> 111.6 mm, vias 6 -> 4
- net /5V: track 72.5 -> 88.2 mm
- net /D2_2: track 2.83 -> 14.7 mm
- net /D7: track 0.00 -> 10.4 mm
- net /D3: track 6.60 -> 14.8 mm
- net /D8: track 0.00 -> 7.80 mm
- net /D4: track 9.51 -> 12.9 mm
- net /GND: track 13.3 -> 16.4 mm
- net /24VS: track 111.8 -> 114.6 mm
- net /D6: track 14.3 -> 11.9 mm
- net /3.3V: track 75.0 -> 76.7 mm, vias 3 -> 4
- net /A2_D0: track 42.6 -> 41.6 mm
- net /D2: track 5.40 -> 6.07 mm

Commit message: Tweaked some pads
Parts:
- moved JP1 3.42 mm to (144.8, 45.7), turned to 0 degrees
- moved J15 2.29 mm to (129.5, 45.7), turned to 0 degrees
Routing:
- net /GND: track 16.4 -> 21.3 mm
- net /5VS: track 111.6 -> 115.2 mm
Changed lines of the file:
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@@
     (thickness 1.6)
     (drawings 5)
-    (tracks 226)
+    (tracks 232)
     (zones 0)
     (modules 32)
@@
   )
   (module Pin_Headers:Pin_Header_Straight_1x02_Pitch2.54mm (layer F.Cu)
-    (at 142.24 48.006 90)
+    (at 144.78 45.72)
     (descr "Through hole straight pin header, 1x02, 2.54mm pitch, single row")
     (tags "Through hole pin header THT 1x02 2.54mm single row")
-    (fp_text reference JP1 (at 0 -2.33 90) (layer F.Fab)
-      (effects (font (size 1 1) (thickness 0.15)))
-    )
-    (fp_text value PRG (at 2.032 2.54 180) (layer F.SilkS)
-      (effects (font (size 1 1) (thickness 0.15)))
-    )
-    (fp_text user %R (at 0 1.27 180) (layer F.Fab)
+    (fp_text reference JP1 (at 0 -2.33) (layer F.Fab)
+      (effects (font (size 1 1) (thickness 0.15)))
+    )
+    (fp_text value PRG (at -2.794 2.54 180) (layer F.SilkS)
+      (effects (font (size 1 1) (thickness 0.15)))
+    )
+    (fp_text user %R (at 0 1.27 90) (layer F.Fab)
       (effects (font (size 1 1) (thickness 0.15)))
     )
@@
     (fp_line (start 1.27 -1.27) (end 1.27 3.81) (layer F.Fab) (width 0.1))
     (fp_line (start -0.635 -1.27) (end 1.27 -1.27) (layer F.Fab) (width 0.1))
-    (pad 2 thru_hole oval (at 0 2.54 90) (size 1.7 1.7) (drill 1) (layers *.Cu *.Mask)
+    (pad 2 thru_hole oval (at 0 2.54) (size 1.7 1.7) (drill 1) (layers *.Cu *.Mask)
       (net 31 /5VS_2))
-    (pad 1 thru_hole rect (at 0 0 90) (size 1.7 1.7) (drill 1) (layers *.Cu *.Mask)
+    (pad 1 thru_hole rect (at 0 0) (size 1.7 1.7) (drill 1) (layers *.Cu *.Mask)
       (net 32 /5VS))
     (model ${KISYS3DMOD}/Pin_Headers.3dshapes/Pin_Header_Straight_1x02_Pitch2.54mm.wrl
@@
   )
   (module Pin_Headers:Pin_Header_Straight_1x02_Pitch2.54mm (layer F.Cu)
-    (at 129.54 48.006 90)
+    (at 129.54 45.72)
     (descr "Through hole straight pin header, 1x02, 2.54mm pitch, single row")
     (tags "Through hole pin header THT 1x02 2.54mm single row")
-    (fp_text reference J15 (at 0 -2.33 90) (layer F.Fab)
-      (effects (font (size 1 1) (thickness 0.15)))
-    )
-    (fp_text value 24S (at 2.032 2.54 180) (layer F.SilkS)
-      (effects (font (size 1 1) (thickness 0.15)))
-    )
-    (fp_text user %R (at 0 1.27 180) (layer F.Fab)
+    (fp_text reference J15 (at 0 -2.33) (layer F.Fab)
+      (effects (font (size 1 1) (thickness 0.15)))
+    )
+    (fp_text value 24S (at 2.794 2.54 180) (layer F.SilkS)
+      (effects (font (size 1 1) (thickness 0.15)))
+    )
+    (fp_text user %R (at 0 1.27 90) (layer F.Fab)
       (effects (font (size 1 1) (thickness 0.15)))
     )
@@
     (fp_line (start 1.27 -1.27) (end 1.27 3.81) (layer F.Fab) (width 0.1))
     (fp_line (start -0.635 -1.27) (end 1.27 -1.27) (layer F.Fab) (width 0.1))
-    (pad 2 thru_hole oval (at 0 2.54 90) (size 1.7 1.7) (drill 1) (layers *.Cu *.Mask)
+    (pad 2 thru_hole oval (at 0 2.54) (size 1.7 1.7) (drill 1) (layers *.Cu *.Mask)
       (net 33 /24VS))
-    (pad 1 thru_hole rect (at 0 0 90) (size 1.7 1.7) (drill 1) (layers *.Cu *.Mask)
+    (pad 1 thru_hole rect (at 0 0) (size 1.7 1.7) (drill 1) (layers *.Cu *.Mask)
       (net 3 /GND))
     (model ${KISYS3DMOD}/Pin_Headers.3dshapes/Pin_Header_Straight_1x02_Pitch2.54mm.wrl
@@
   (segment (start 150.622 110.744) (end 149.606 111.76) (width 0.2032) (layer F.Cu) (net 2))
   (segment (start 129.286 53.086) (end 129.54 53.34) (width 0.3048) (layer F.Cu) (net 3))
-  (segment (start 129.54 48.006) (end 129.54 53.086) (width 0.3048) (layer F.Cu) (net 3))
   (segment (start 141.146 100.33) (end 152.146 100.33) (width 0.3048) (layer B.Cu) (net 3))
+  (segment (start 130.6948 45.72) (end 131.572 46.5972) (width 0.3048) (layer F.Cu) (net 3))
+  (segment (start 129.54 45.72) (end 130.6948 45.72) (width 0.3048) (layer F.Cu) (net 3))
+  (segment (start 129.54 52.2352) (end 129.54 53.34) (width 0.3048) (layer F.Cu) (net 3))
+  (segment (start 131.572 50.2032) (end 129.54 52.2352) (width 0.3048) (layer F.Cu) (net 3))
+  (segment (start 131.572 46.5972) (end 131.572 50.2032) (width 0.3048) (layer F.Cu) (net 3))
   (segment (start 133.096 104.394) (end 133.096 100.838) (width 0.2032) (layer F.Cu) (net 4))
   (segment (start 134.874 106.172) (end 133.096 104.394) (width 0.2032) (layer F.Cu) (net 4))
@@
   (segment (start 142.24 89.662) (end 142.748 89.154) (width 0.3048) (layer F.Cu) (net 30))
   (segment (start 144.78 53.34) (end 145.288 53.34) (width 0.3048) (layer F.Cu) (net 31))
-  (segment (start 144.78 53.34) (end 144.78 48.006) (width 0.3048) (layer F.Cu) (net 31))
+  (segment (start 144.78 48.26) (end 144.78 53.34) (width 0.3048) (layer F.Cu) (net 31))
   (via (at 152.146 97.79) (size 0.6858) (drill 0.3302) (layers F.Cu B.Cu) (net 32))
   (segment (start 123.1 104.92) (end 123.1 104.6) (width 0.3048) (layer F.Cu) (net 32))
   (segment (start 123.1 104.92) (end 125.494 104.92) (width 2.54) (layer F.Cu) (net 32))
-  (segment (start 142.748 66.294) (end 142.748 48.514) (width 0.3048) (layer F.Cu) (net 32))
-  (segment (start 142.748 48.514) (end 142.24 48.006) (width 0.3048) (layer F.Cu) (net 32))
   (via (at 142.748 66.294) (size 0.6858) (drill 0.3302) (layers F.Cu B.Cu) (net 32))
   (via (at 142.748 70.612) (size 0.6858) (drill 0.3302) (layers F.Cu B.Cu) (net 32))
@@
   (segment (start 137.922 98.552) (end 136.906 99.568) (width 2.54) (layer F.Cu) (net 32))
   (segment (start 137.922 95.25) (end 137.922 98.552) (width 2.54) (layer F.Cu) (net 32))
+  (segment (start 143.6252 45.72) (end 144.78 45.72) (width 0.3048) (layer F.Cu) (net 32))
+  (segment (start 142.748 46.5972) (end 143.6252 45.72) (width 0.3048) (layer F.Cu) (net 32))
+  (segment (start 142.748 66.294) (end 142.748 46.5972) (width 0.3048) (layer F.Cu) (net 32))
   (segment (start 124.42 53.3) (end 124.46 53.34) (width 1.905) (layer F.Cu) (net 33))
   (segment (start 124.46 53.34) (end 123.444 53.34) (width 2.54) (layer B.Cu) (net 33))
@@
   (segment (start 149.8 52.832) (end 147.768 50.8) (width 2.54) (layer B.Cu) (net 33))
   (segment (start 149.8 53.34) (end 149.8 52.832) (width 2.54) (layer B.Cu) (net 33))
-  (segment (start 132.08 48.006) (end 132.08 50.8) (width 2.54) (layer B.Cu) (net 33))
-  (segment (start 126.492 50.8) (end 131.826 50.8) (width 2.54) (layer B.Cu) (net 33))
   (segment (start 131.826 50.8) (end 147.768 50.8) (width 2.54) (layer B.Cu) (net 33))
+  (segment (start 129.54 48.26) (end 129.54 50.8) (width 2.54) (layer B.Cu) (net 33))
+  (segment (start 126.492 50.8) (end 129.54 50.8) (width 2.54) (layer B.Cu) (net 33))
+  (segment (start 129.54 50.8) (end 131.826 50.8) (width 2.54) (layer B.Cu) (net 33))
   (segment (start 136.84 119.4) (end 136.86 119.42) (width 0.2032) (layer F.Cu) (net 34))
   (segment (start 136.886 119.4) (end 136.906 119.38) (width 0.2032) (layer F.Cu) (net 34))

Commit message: Small tweaks
Parts:
- J15: value 24S -> 24VS
Changed lines of the file:
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@@
       (effects (font (size 1 1) (thickness 0.15)))
     )
-    (fp_text value 24S (at 2.794 2.54 180) (layer F.SilkS)
+    (fp_text value 24VS (at 3.302 2.54 180) (layer F.SilkS)
       (effects (font (size 1 1) (thickness 0.15)))
     )
