File: schematic/main/main.sch (KiCad schematic (older format))
At the start: 17 parts, among them J1 Button, J2 Sensor, J3 5V Relay, J4 24V Relay, J5 LEDs, J6 Fan, M1 LLC4, T1 5V, T2 5VS, T3 24VS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

Commit message: PCBs started!
Parts:
- added JP1: PRG, Pin_Headers:Pin_Header_Straight_1x02_Pitch2.54mm, symbol Device:Jumper
- A1: footprint Module:Arduino_Pro_Mini -> arduino_pro_mini:arduino_pro_mini
- A2: footprint Module:Teensy_32 -> teensy_32:teensy_32
- C1: footprint (none) -> Capacitors_THT:CP_Radial_D12.5mm_P5.00mm
- CON1: renamed from JP2; value Right Pumps -> Left Pumps; footprint (none) -> Pin_Headers:Pin_Header_Angled_1x15_Pitch2.54mm
- CON2: renamed from JP1; value Left Pumps -> Right Pumps; footprint (none) -> Pin_Headers:Pin_Header_Angled_1x15_Pitch2.54mm
- J1, J6: footprint (none) -> Pin_Headers:Pin_Header_Straight_1x02_Pitch2.54mm
- J2, J3, J4, J5: footprint (none) -> Pin_Headers:Pin_Header_Straight_1x03_Pitch2.54mm
- M1: footprint LLC4 -> logic_level_converter:LLC4
- R1: footprint (none) -> Resistors_THT:R_Axial_DIN0309_L9.0mm_D3.2mm_P2.54mm_Vertical
- T1, T2, T3, T4: footprint (none) -> Wire_Pads:SolderWirePad_2x_1-5mmDrill
Connections:
- net 3.3V: now also CON1.8 (Pin_8), CON2.8 (Pin_8)
- net 5VS: now also JP1.1; no longer A2.33 (VIN), CON1.8 (Pin_8), CON2.8 (Pin_8)
- net A1_D0: now also M1.7 (HL4); no longer M1.11 (HL2)
- net A1_D1: now also M1.8 (HL3); no longer M1.12 (HL4)
- net A2_D0: now also M1.5 (LV3); no longer M1.1 (LV1)
- net A2_D1: now also M1.6 (LV4); no longer M1.2 (LV2)
- net DIR: now also A2.12 (D10); no longer A2.27 (D20/A6)
- net GND: now also CON1.2 (Pin_2), CON2.2 (Pin_2)
- net P0: now also A2.30 (D23/A9), CON1.3 (Pin_3); no longer A2.4 (D2), CON2.3 (Pin_3)
- net P1: now also A2.29 (D22/A8), CON1.4 (Pin_4); no longer A2.5 (D3), CON2.4 (Pin_4)
- net P10: now also A2.9 (D7), CON2.5 (Pin_5); no longer A2.14 (D12), CON1.11 (Pin_11)
- net P11: now also A2.8 (D6), CON2.6 (Pin_6); no longer A2.21 (D14/A0), CON1.10 (Pin_10)
- net P12: now also A2.7 (D5), CON2.10 (Pin_10); no longer A2.22 (D15/A1), CON1.6 (Pin_6)
- net P13: now also A2.6 (D4), CON2.11 (Pin_11); no longer A2.23 (D16/A2), CON1.5 (Pin_5)
- net P14: now also A2.5 (D3), CON2.12 (Pin_12); no longer A2.24 (D17/A3), CON1.4 (Pin_4)
- net P15: now also A2.4 (D2), CON2.13 (Pin_13); no longer A2.25 (D18/A4), CON1.3 (Pin_3)
- net P2: now also A2.28 (D21/A7), CON1.5 (Pin_5); no longer A2.6 (D4), CON2.5 (Pin_5)
- net P3: now also A2.27 (D20/A6), CON1.6 (Pin_6); no longer A2.7 (D5), CON2.6 (Pin_6)
- net P4: now also A2.26 (D19/A5), CON1.10 (Pin_10); no longer A2.8 (D6), CON2.10 (Pin_10)
- net P5: now also A2.25 (D18/A4), CON1.11 (Pin_11); no longer A2.9 (D7), CON2.11 (Pin_11)
- net P6: now also A2.24 (D17/A3), CON1.12 (Pin_12); no longer A2.10 (D8), CON2.12 (Pin_12)
- net P7: now also A2.23 (D16/A2), CON1.13 (Pin_13); no longer A2.11 (D9), CON2.13 (Pin_13)
- net P8: now also A2.11 (D9), CON2.3 (Pin_3); no longer A2.12 (D10), CON1.13 (Pin_13)
- net P9: now also A2.10 (D8), CON2.4 (Pin_4); no longer A2.13 (D11), CON1.12 (Pin_12)
- net ~ENABLE: now also A2.13 (D11); no longer A2.26 (D19/A5)
- new net 5VS_2: A2.33 (VIN), JP1.2

Commit message: Finished board designs.
Parts:
- removed T1: 5V, Wire_Pads:SolderWirePad_2x_1-5mmDrill, symbol Connector:Conn_01x01_Male
- removed T2: 5VS, Wire_Pads:SolderWirePad_2x_1-5mmDrill, symbol Connector:Conn_01x01_Male
- removed T3: 24VS, Wire_Pads:SolderWirePad_2x_1-5mmDrill, symbol Connector:Conn_01x01_Male
- removed T4: GND, Wire_Pads:SolderWirePad_2x_1-5mmDrill, symbol Connector:Conn_01x01_Male
- added J7: Pi, Pin_Headers:Pin_Header_Straight_1x02_Pitch2.54mm, symbol Connector:Conn_01x02_Male
- added T1: 5V, spade_terminal:Spade_Terminal_1_4, symbol spade_terminal:Spade_Terminal
- added T2: 5VS, spade_terminal:Spade_Terminal_1_4, symbol spade_terminal:Spade_Terminal
- added T3: 24VS, spade_terminal:Spade_Terminal_1_4, symbol spade_terminal:Spade_Terminal
- added T4: GND, spade_terminal:Spade_Terminal_1_4, symbol spade_terminal:Spade_Terminal
- CON1: value Left Pumps -> Left
- CON2: value Right Pumps -> Right
- R1: footprint Resistors_THT:R_Axial_DIN0309_L9.0mm_D3.2mm_P2.54mm_Vertical -> Resistors_THT:R_Axial_DIN0207_L6.3mm_D2.5mm_P2.54mm_Vertical
Connections:
- net 24VS: now also T3.1 (Pin_1); no longer J6.1 (Pin_1)
- net 5V: now also J3.3 (Pin_3), J4.3 (Pin_3), T1.1 (Pin_1); no longer J3.1 (Pin_1), J4.1 (Pin_1)
- net 5VS: now also J5.3 (Pin_3), J6.2 (Pin_2), J7.2 (Pin_2), T2.1 (Pin_1); no longer J5.1 (Pin_1)
- net A1_D0: now also M1.11 (HL2); no longer M1.7 (HL4)
- net A1_D1: now also M1.12 (HL4); no longer M1.8 (HL3)
- net A2_D0: now also M1.1 (LV1); no longer M1.5 (LV3)
- net A2_D1: now also M1.2 (LV2); no longer M1.6 (LV4)
- net D2: now also J5.2 (Pin_2), R1.1; no longer A1.5 (D2), J1.1 (Pin_1)
- net D3: now also J2.3 (Pin_3); no longer J2.1 (Pin_1)
- net D4: now also J1.2 (Pin_2); no longer J3.2 (Pin_2)
- net D5: now also J3.2 (Pin_2); no longer J4.2 (Pin_2)
- net D6: now also J4.2 (Pin_2); no longer R1.1
- net GND: now also J1.1 (Pin_1), J2.1 (Pin_1), J3.1 (Pin_1), J4.1 (Pin_1), J5.1 (Pin_1), J6.1 (Pin_1), J7.1 (Pin_1), T4.1 (Pin_1); no longer J1.2 (Pin_2), J2.3 (Pin_3), J3.3 (Pin_3), J4.3 (Pin_3), J5.3 (Pin_3), J6.2 (Pin_2)
- net D2_2: now reaches R1.2
- net D2_2: now also A1.5 (D2); no longer J5.2 (Pin_2)
Other:
- moved on the sheet: J1, J3, J4, J5, J6, R1

Commit message: Tweaked schematic and board
Parts:
- added J10, J11: 5VS, Pin_Headers:Pin_Header_Straight_1x02_Pitch2.54mm, symbol Connector:Conn_01x02_Male
- added J12, J13, J14: 5V, Pin_Headers:Pin_Header_Straight_1x02_Pitch2.54mm, symbol Connector:Conn_01x02_Male
- added J15: 24S, Pin_Headers:Pin_Header_Straight_1x02_Pitch2.54mm, symbol Connector:Conn_01x02_Male
- added J16: 3.3V, Pin_Headers:Pin_Header_Straight_1x02_Pitch2.54mm, symbol Connector:Conn_01x02_Male
- added J2: Sensor0, Pin_Headers:Pin_Header_Straight_1x03_Pitch2.54mm, symbol Connector:Conn_01x03_Male
- added J6: Relay2, Pin_Headers:Pin_Header_Straight_1x03_Pitch2.54mm, symbol Connector:Conn_01x03_Male
- C1: footprint Capacitors_THT:CP_Radial_D12.5mm_P5.00mm -> Capacitors_THT:CP_Radial_D10.0mm_P5.00mm
- J3: renamed from J2; value Sensor -> Sensor1
- J4: renamed from J3; value 5V Relay -> Relay0
- J5: renamed from J4; value 24V Relay -> Relay1
- J8: renamed from J6; value Fan -> 5VS
- J9: renamed from J7; value Pi -> 5VS
- renumbered J5 to J1, J1 to J7
Connections:
- net 24VS: now also J15.2 (Pin_2)
- net 3.3V: now also J16.2 (Pin_2)
- net 5V: now also C1.1, J12.2 (Pin_2), J13.2 (Pin_2), J14.2 (Pin_2), J6.3 (Pin_3)
- net 5VS: now also J10.2 (Pin_2), J11.2 (Pin_2), J2.2 (Pin_2); no longer C1.1
- net D3: now also J2.3 (Pin_3); no longer J3.3 (Pin_3)
- net D4: now also J3.3 (Pin_3); no longer J7.2 (Pin_2)
- net GND: now also J10.1 (Pin_1), J11.1 (Pin_1), J12.1 (Pin_1), J13.1 (Pin_1), J14.1 (Pin_1), J15.1 (Pin_1), J16.1 (Pin_1), J2.1 (Pin_1), J6.1 (Pin_1)
- net D7: now reaches A1.10 (D7)
- net D7: now also J6.2 (Pin_2)
- net D8: now reaches A1.11 (D8)
- net D8: now also J7.2 (Pin_2)
- no-connect marks 33 -> 31
Other:
- moved on the sheet: C1, J1, J4, J5, J7, R1, T1, T2, T4

Commit message: No real changes
Parts:
- C1: symbol Device:CP1 -> main-rescue:CP1-Device-main-rescue
- CON1, CON2: symbol Connector:Conn_01x15_Male -> main-rescue:Conn_01x15_Male-Connector-main-rescue
- J1, J2, J3, J4, J5, J6: symbol Connector:Conn_01x03_Male -> main-rescue:Conn_01x03_Male-Connector-main-rescue
- J10, J11, J12, J13, J14, J15, J16, J7, J8, J9: symbol Connector:Conn_01x02_Male -> main-rescue:Conn_01x02_Male-Connector-main-rescue
- JP1: symbol Device:Jumper -> main-rescue:Jumper-Device-main-rescue
- R1: symbol Device:R_US -> main-rescue:R_US-Device-main-rescue
Changed lines of the file:
@@
 $EndComp
 $Comp
-L Connector:Conn_01x03_Male J3
+L main-rescue:Conn_01x03_Male-Connector-main-rescue J3
 U 1 1 5BCF834E
 P 1150 2650
@@
 $EndComp
 $Comp
-L Connector:Conn_01x02_Male J7
+L main-rescue:Conn_01x02_Male-Connector-main-rescue J7
 U 1 1 5BCF83FD
 P 1150 4500
@@
 $EndComp
 $Comp
-L Connector:Conn_01x03_Male J4
+L main-rescue:Conn_01x03_Male-Connector-main-rescue J4
 U 1 1 5BCF8720
 P 1150 3150
@@
 $EndComp
 $Comp
-L Connector:Conn_01x03_Male J5
+L main-rescue:Conn_01x03_Male-Connector-main-rescue J5
 U 1 1 5BCF8793
 P 1150 3600
@@
 $EndComp
 $Comp
-L Device:R_US R1
+L main-rescue:R_US-Device-main-rescue R1
 U 1 1 5BCF9849
 P 2350 1900
@@
 $EndComp
 $Comp
-L Device:CP1 C1
+L main-rescue:CP1-Device-main-rescue C1
 U 1 1 5BCF98F0
 P 4200 3000
@@
 Connection ~ 3200 3800
 $Comp
-L Connector:Conn_01x03_Male J1
+L main-rescue:Conn_01x03_Male-Connector-main-rescue J1
 U 1 1 5BCFDB4F
 P 1150 1700
@@
 	5500 5100 5500 4400
 $Comp
-L power:PWR_FLAG #FLG0101
+L main-rescue:PWR_FLAG-power-main-rescue #FLG0101
 U 1 1 5BE4B784
 P 2850 7000
@@
 	2850 7000 3200 7000
 $Comp
-L power:PWR_FLAG #FLG0102
+L main-rescue:PWR_FLAG-power-main-rescue #FLG0102
 U 1 1 5BE4B7FF
 P 2500 1200
@@
 $EndComp
 $Comp
-L power:PWR_FLAG #FLG0103
+L main-rescue:PWR_FLAG-power-main-rescue #FLG0103
 U 1 1 5BE4B85A
 P 2500 900
@@
 DIR
 $Comp
-L Connector:Conn_01x02_Male J8
+L main-rescue:Conn_01x02_Male-Connector-main-rescue J8
 U 1 1 5BE5E3EF
 P 1150 5500
@@
 	5950 5350 6400 5350
 $Comp
-L Connector:Conn_01x15_Male CON2
+L main-rescue:Conn_01x15_Male-Connector-main-rescue CON2
 U 1 1 5BCFD97B
 P 5750 5550
@@
 $EndComp
 $Comp
-L Connector:Conn_01x15_Male CON1
+L main-rescue:Conn_01x15_Male-Connector-main-rescue CON1
 U 1 1 5BCFD9D4
 P 9550 5550
@@
 	6000 1500 7800 1500
 $Comp
-L Device:Jumper JP1
+L main-rescue:Jumper-Device-main-rescue JP1
 U 1 1 5BD13E35
 P 6200 1300
@@
 	5900 1300 4950 1300
 $Comp
-L power:PWR_FLAG #FLG0104
+L main-rescue:PWR_FLAG-power-main-rescue #FLG0104
 U 1 1 5BD2178B
 P 7350 1300
@@
 	1350 5100 2300 5100
 $Comp
-L Connector:Conn_01x02_Male J9
+L main-rescue:Conn_01x02_Male-Connector-main-rescue J9
 U 1 1 5BD40086
 P 1150 5900
@@
 NoConn ~ 5400 2300
 $Comp
-L Connector:Conn_01x02_Male J10
+L main-rescue:Conn_01x02_Male-Connector-main-rescue J10
 U 1 1 5BD7937E
 P 1150 6250
@@
 Connection ~ 1650 6000
 $Comp
-L Connector:Conn_01x03_Male J2
+L main-rescue:Conn_01x03_Male-Connector-main-rescue J2
 U 1 1 5BD94D86
 P 1150 2200
@@
 	1550 7000 2850 7000
 $Comp
-L Connector:Conn_01x03_Male J6
+L main-rescue:Conn_01x03_Male-Connector-main-rescue J6
 U 1 1 5BF25C51
 P 1150 4050
@@
 D8
 $Comp
-L Connector:Conn_01x02_Male J11
+L main-rescue:Conn_01x02_Male-Connector-main-rescue J11
 U 1 1 5BF738A8
 P 1150 6600
@@
 Connection ~ 1650 6350
 $Comp
-L Connector:Conn_01x02_Male J12
+L main-rescue:Conn_01x02_Male-Connector-main-rescue J12
 U 1 1 5BFFDCD1
 P 2150 5500
@@
 $EndComp
 $Comp
-L Connector:Conn_01x02_Male J13
+L main-rescue:Conn_01x02_Male-Connector-main-rescue J13
 U 1 1 5C043D16
 P 2150 5900
@@
 $EndComp
 $Comp
-L Connector:Conn_01x02_Male J14
+L main-rescue:Conn_01x02_Male-Connector-main-rescue J14
 U 1 1 5C043D64
 P 2150 6250
@@
 Connection ~ 1750 6000
 $Comp
-L Connector:Conn_01x02_Male J15
+L main-rescue:Conn_01x02_Male-Connector-main-rescue J15
 U 1 1 5C0A867B
 P 2650 6600
@@
 	2300 5100 5500 5100
 $Comp
-L Connector:Conn_01x02_Male J16
+L main-rescue:Conn_01x02_Male-Connector-main-rescue J16
 U 1 1 5C0D0641
 P 2550 5500
