File: schematic/pump/module.sch (KiCad schematic (older format))
At the start: 3 parts, among them J1 Motor

Commit message: PCBs started!
Parts:
- A1: footprint Module:DRV8825_Carrier -> Modules:Pololu_Breakout-16_15.2x20.3mm
- C1: footprint (none) -> Capacitors_THT:CP_Radial_D6.3mm_P2.50mm
- J1: footprint (none) -> Pin_Headers:Pin_Header_Straight_1x04_Pitch2.54mm
Connections:
- net A2: now reaches A1.11 (A2), J1.4 (Pin_4)
- net A1: now reaches A1.12 (A1), J1.3 (Pin_3)
- net B1: now reaches A1.13 (B1), J1.2 (Pin_2)
- net B2: now reaches A1.14 (B2), J1.1 (Pin_1)
- net M2: now reaches A1.4 (M2)
- net 3.3V: now reaches A1.5 (~RESET)
- net 3.3V: now also A1.6 (~SLEEP)
- net 5V renamed M0
- net M0: no longer A1.3 (M1)
- new net M1: A1.3 (M1)
- no-connect marks 4 -> 1
Changed lines of the file:
@@
 $Descr A4 11693 8268
 encoding utf-8
-Sheet 9 9
+Sheet 3 9
 Title ""
 Date ""
@@
 AR Path="/5BCF8E81/5BCF6E5D" Ref="A6"  Part="1"
 AR Path="/5BCF8E85/5BCF6E5D" Ref="A7"  Part="1"
-F 0 "A7" H 5350 4450 50  0000 C CNN
+AR Path="/5BCF6D72/5BCF6E5D" Ref="A0"  Part="1"
+F 0 "A3" H 5350 4450 50  0000 C CNN
 F 1 "DRV8825_Carrier" H 6150 4450 50  0000 C CNN
-F 2 "Module:DRV8825_Carrier" H 5850 2950 50  0001 L CNN
+F 2 "Modules:Pololu_Breakout-16_15.2x20.3mm" H 5850 2950 50  0001 L CNN
 F 3 "https://www.pololu.com/product/2133" H 5500 4550 50  0001 C CNN
 	1    5700 3700
@@
 AR Path="/5BCF8E81/5BCF6EE0" Ref="C6"  Part="1"
 AR Path="/5BCF8E85/5BCF6EE0" Ref="C7"  Part="1"
-F 0 "C7" V 4715 4546 50  0000 L CNN
+AR Path="/5BCF6D72/5BCF6EE0" Ref="C0"  Part="1"
+F 0 "C3" V 4715 4546 50  0000 L CNN
 F 1 "100u" H 4715 4455 50  0000 L CNN
-F 2 "" H 4600 4500 50  0001 C CNN
+F 2 "Capacitors_THT:CP_Radial_D6.3mm_P2.50mm" H 4600 4500 50  0001 C CNN
 F 3 "~" H 4600 4500 50  0001 C CNN
 	1    4600 4500
@@
 AR Path="/5BCF8E81/5BCF6FDD" Ref="J6"  Part="1"
 AR Path="/5BCF8E85/5BCF6FDD" Ref="J7"  Part="1"
-F 0 "J7" H 6672 3373 50  0000 R CNN
+AR Path="/5BCF6D72/5BCF6FDD" Ref="J0"  Part="1"
+F 0 "J3" H 6672 3373 50  0000 R CNN
 F 1 "Motor" H 6672 3282 50  0000 R CNN
-F 2 "" H 6700 3400 50  0001 C CNN
+F 2 "Pin_Headers:Pin_Header_Straight_1x04_Pitch2.54mm" H 6700 3400 50  0001 C CNN
 F 3 "~" H 6700 3400 50  0001 C CNN
 	1    6700 3400
@@
 Wire Wire Line
 	3700 3300 5200 3300
-NoConn ~ 5200 3400
-NoConn ~ 5200 3500
 Wire Wire Line
 	3700 2650 4600 2650
@@
 Wire Wire Line
 	3700 4100 5200 4100
-Wire Wire Line
-	5200 3700 5100 3700
-Wire Wire Line
-	5100 3700 5100 3800
-Wire Wire Line
-	5100 3800 5200 3800
-NoConn ~ 5200 3900
 NoConn ~ 6200 3800
-Text HLabel 3700 3700 0    50   Input ~ 0
-5V
-Wire Wire Line
-	3700 3700 5100 3700
-Connection ~ 5100 3700
+Text HLabel 3700 3400 0    50   Input ~ 0
+3.3V
 Wire Wire Line
 	6200 3300 6500 3300
@@
 Wire Wire Line
 	6200 3600 6500 3600
+Wire Wire Line
+	3700 3400 5100 3400
+Wire Wire Line
+	5100 3400 5100 3500
+Wire Wire Line
+	5100 3500 5200 3500
+Connection ~ 5100 3400
+Wire Wire Line
+	5100 3400 5200 3400
+Wire Wire Line
+	3700 3700 5200 3700
+Text HLabel 3700 3700 0    50   Input ~ 0
+M0
+Text HLabel 3700 3800 0    50   Input ~ 0
+M1
+Text HLabel 3700 3900 0    50   Input ~ 0
+M2
+Wire Wire Line
+	3700 3800 5200 3800
+Wire Wire Line
+	3700 3900 5200 3900
+Text Label 6350 3300 0    50   ~ 0
+B2
+Text Label 6350 3400 0    50   ~ 0
+B1
+Text Label 6350 3500 0    50   ~ 0
+A1
+Text Label 6350 3600 0    50   ~ 0
+A2
 $EndSCHEMATC

Commit message: Finished board designs.
Connections:
- net A1: now also J1.2 (Pin_2); no longer J1.3 (Pin_3)
- net A2: now also J1.1 (Pin_1); no longer J1.4 (Pin_4)
- net B1: now also J1.3 (Pin_3); no longer J1.2 (Pin_2)
- net B2: now also J1.4 (Pin_4); no longer J1.1 (Pin_1)
Changed lines of the file:
@@
 AR Path="/5BCF8E85/5BCF6E5D" Ref="A7"  Part="1"
 AR Path="/5BCF6D72/5BCF6E5D" Ref="A0"  Part="1"
-F 0 "A3" H 5350 4450 50  0000 C CNN
+F 0 "A1" H 5350 4450 50  0000 C CNN
 F 1 "DRV8825_Carrier" H 6150 4450 50  0000 C CNN
 F 2 "Modules:Pololu_Breakout-16_15.2x20.3mm" H 5850 2950 50  0001 L CNN
@@
 AR Path="/5BCF8E85/5BCF6EE0" Ref="C7"  Part="1"
 AR Path="/5BCF6D72/5BCF6EE0" Ref="C0"  Part="1"
-F 0 "C3" V 4715 4546 50  0000 L CNN
+F 0 "C1" V 4715 4546 50  0000 L CNN
 F 1 "100u" H 4715 4455 50  0000 L CNN
 F 2 "Capacitors_THT:CP_Radial_D6.3mm_P2.50mm" H 4600 4500 50  0001 C CNN
@@
 L Connector:Conn_01x04_Male J1
 U 1 1 5BCF6FDD
-P 6700 3400
+P 6700 3500
 AR Path="/5BCF8DAA/5BCF6FDD" Ref="J1"  Part="1"
 AR Path="/5BCF8E71/5BCF6FDD" Ref="J2"  Part="1"
@@
 AR Path="/5BCF8E85/5BCF6FDD" Ref="J7"  Part="1"
 AR Path="/5BCF6D72/5BCF6FDD" Ref="J0"  Part="1"
-F 0 "J3" H 6672 3373 50  0000 R CNN
-F 1 "Motor" H 6672 3282 50  0000 R CNN
-F 2 "Pin_Headers:Pin_Header_Straight_1x04_Pitch2.54mm" H 6700 3400 50  0001 C CNN
-F 3 "~" H 6700 3400 50  0001 C CNN
-	1    6700 3400
-	-1   0    0    -1
+F 0 "J1" H 6672 3473 50  0000 R CNN
+F 1 "Motor" H 6672 3382 50  0000 R CNN
+F 2 "Pin_Headers:Pin_Header_Straight_1x04_Pitch2.54mm" H 6700 3500 50  0001 C CNN
+F 3 "~" H 6700 3500 50  0001 C CNN
+	1    6700 3500
+	-1   0    0    1
 $EndComp
 Text HLabel 3700 3300 0    50   Input ~ 0

Commit message: No real changes
Parts:
- C1: symbol Device:CP1 -> pump-rescue:CP1-Device
- J1: symbol Connector:Conn_01x04_Male -> pump-rescue:Conn_01x04_Male-Connector
Changed lines of the file:
@@
 $EndComp
 $Comp
-L Device:CP1 C1
+L pump-rescue:CP1-Device C1
 U 1 1 5BCF6EE0
 P 4600 4500
@@
 AR Path="/5BCF8E85/5BCF6EE0" Ref="C7"  Part="1"
 AR Path="/5BCF6D72/5BCF6EE0" Ref="C0"  Part="1"
+AR Path="/5BCF6EE0" Ref="C1"  Part="1"
 F 0 "C1" V 4715 4546 50  0000 L CNN
 F 1 "100u" H 4715 4455 50  0000 L CNN
@@
 $EndComp
 $Comp
-L Connector:Conn_01x04_Male J1
+L pump-rescue:Conn_01x04_Male-Connector J1
 U 1 1 5BCF6FDD
 P 6700 3500
@@
 AR Path="/5BCF8E85/5BCF6FDD" Ref="J7"  Part="1"
 AR Path="/5BCF6D72/5BCF6FDD" Ref="J0"  Part="1"
+AR Path="/5BCF6FDD" Ref="J1"  Part="1"
 F 0 "J1" H 6672 3473 50  0000 R CNN
 F 1 "Motor" H 6672 3382 50  0000 R CNN
