File: schematic/pump/pump.sch (KiCad schematic (older format))
At the start: 1 part

Commit message: PCBs started!
Parts:
- added JP1: M0, Pin_Headers:Pin_Header_Straight_2x01_Pitch2.54mm, symbol Device:Jumper_NC_Small
- added JP2: M1, Pin_Headers:Pin_Header_Straight_2x01_Pitch2.54mm, symbol Device:Jumper_NC_Small
- added JP3: M2, Pin_Headers:Pin_Header_Straight_2x01_Pitch2.54mm, symbol Device:Jumper_NC_Small
- CON1: renamed from H1; footprint (none) -> Socket_Strips:Socket_Strip_Angled_1x15_Pitch2.54mm
Connections:
- net 5V renamed 3.3V
- net 3.3V: now also JP1.2, JP2.2, JP3.2
- new net M0: JP1.1
- new net M1: JP2.1
- new net M2: JP3.1
Changed lines of the file:
@@
 F5 "24V" I L 4150 1450 50
 F6 "GND" I L 4150 1650 50
-F7 "5V" I L 4150 1550 50
+F7 "3.3V" I L 4150 1550 50
+F8 "M0" I R 4750 1250 50
+F9 "M1" I R 4750 1350 50
+F10 "M2" I R 4750 1450 50
 $EndSheet
 $Comp
-L Connector:Conn_01x15_Female H1
+L Connector:Conn_01x15_Female CON1
 U 1 1 5BCF8B18
 P 1750 4550
-F 0 "H1" H 1650 5400 50  0000 C CNN
+F 0 "CON1" H 1650 5400 50  0000 C CNN
 F 1 "Main" H 1650 3750 50  0000 C CNN
-F 2 "" H 1750 4550 50  0001 C CNN
+F 2 "Socket_Strips:Socket_Strip_Angled_1x15_Pitch2.54mm" H 1750 4550 50  0001 C CNN
 F 3 "~" H 1750 4550 50  0001 C CNN
 	1    1750 4550
@@
 F5 "24V" I L 4150 2350 50
 F6 "GND" I L 4150 2550 50
-F7 "5V" I L 4150 2450 50
+F7 "3.3V" I L 4150 2450 50
+F8 "M0" I R 4750 2150 50
+F9 "M1" I R 4750 2250 50
+F10 "M2" I R 4750 2350 50
 $EndSheet
 $Sheet
@@
 F5 "24V" I L 4150 3250 50
 F6 "GND" I L 4150 3450 50
-F7 "5V" I L 4150 3350 50
+F7 "3.3V" I L 4150 3350 50
+F8 "M0" I R 4750 3050 50
+F9 "M1" I R 4750 3150 50
+F10 "M2" I R 4750 3250 50
 $EndSheet
 $Sheet
@@
 F5 "24V" I L 4150 4150 50
 F6 "GND" I L 4150 4350 50
-F7 "5V" I L 4150 4250 50
+F7 "3.3V" I L 4150 4250 50
+F8 "M0" I R 4750 3950 50
+F9 "M1" I R 4750 4050 50
+F10 "M2" I R 4750 4150 50
 $EndSheet
 $Sheet
@@
 F5 "24V" I L 4150 5050 50
 F6 "GND" I L 4150 5250 50
-F7 "5V" I L 4150 5150 50
+F7 "3.3V" I L 4150 5150 50
+F8 "M0" I R 4750 4850 50
+F9 "M1" I R 4750 4950 50
+F10 "M2" I R 4750 5050 50
 $EndSheet
 $Sheet
@@
 F5 "24V" I L 4150 5950 50
 F6 "GND" I L 4150 6150 50
-F7 "5V" I L 4150 6050 50
+F7 "3.3V" I L 4150 6050 50
+F8 "M0" I R 4750 5750 50
+F9 "M1" I R 4750 5850 50
+F10 "M2" I R 4750 5950 50
 $EndSheet
 $Sheet
@@
 F5 "24V" I L 4150 6900 50
 F6 "GND" I L 4150 7100 50
-F7 "5V" I L 4150 7000 50
+F7 "3.3V" I L 4150 7000 50
+F8 "M0" I R 4750 6700 50
+F9 "M1" I R 4750 6800 50
+F10 "M2" I R 4750 6900 50
 $EndSheet
 $Sheet
@@
 F5 "24V" I L 4150 7850 50
 F6 "GND" I L 4150 8050 50
-F7 "5V" I L 4150 7950 50
+F7 "3.3V" I L 4150 7950 50
+F8 "M0" I R 4750 7650 50
+F9 "M1" I R 4750 7750 50
+F10 "M2" I R 4750 7850 50
 $EndSheet
 Wire Wire Line
@@
 ~ENABLE
 Text Label 2500 4550 0    50   ~ 0
-5V
+3.3V
 Text Label 2500 4650 0    50   ~ 0
 DIR
@@
 Wire Wire Line
 	3100 3950 3600 3950
+Wire Wire Line
+	4750 1250 4900 1250
+Wire Wire Line
+	4900 1250 4900 2150
+Wire Wire Line
+	4900 2150 4750 2150
+Wire Wire Line
+	4900 2150 4900 3050
+Wire Wire Line
+	4900 3050 4750 3050
+Connection ~ 4900 2150
+Wire Wire Line
+	4900 3050 4900 3950
+Wire Wire Line
+	4900 3950 4750 3950
+Connection ~ 4900 3050
+Wire Wire Line
+	4900 3950 4900 4850
+Wire Wire Line
+	4900 4850 4750 4850
+Connection ~ 4900 3950
+Wire Wire Line
+	4900 4850 4900 5750
+Wire Wire Line
+	4900 5750 4750 5750
+Connection ~ 4900 4850
+Wire Wire Line
+	4750 1350 5000 1350
+Wire Wire Line
+	5000 1350 5000 2250
+Wire Wire Line
+	5000 2250 4750 2250
+Wire Wire Line
+	5000 2250 5000 3150
+Wire Wire Line
+	5000 3150 4750 3150
+Connection ~ 5000 2250
+Wire Wire Line
+	5000 3150 5000 4050
+Wire Wire Line
+	5000 4050 4750 4050
+Connection ~ 5000 3150
+Wire Wire Line
+	5000 4050 5000 4950
+Wire Wire Line
+	5000 4950 4750 4950
+Connection ~ 5000 4050
+Wire Wire Line
+	5000 4950 5000 5850
+Wire Wire Line
+	5000 5850 4750 5850
+Connection ~ 5000 4950
+Wire Wire Line
+	4750 1450 5100 1450
+Wire Wire Line
+	5100 1450 5100 2350
+Wire Wire Line
+	5100 2350 4750 2350
+Wire Wire Line
+	5100 2350 5100 3250
+Wire Wire Line
+	5100 3250 4750 3250
+Connection ~ 5100 2350
+Wire Wire Line
+	5100 3250 5100 4150
+Wire Wire Line
+	5100 4150 4750 4150
+Connection ~ 5100 3250
+Wire Wire Line
+	5100 4150 5100 5050
+Wire Wire Line
+	5100 5050 4750 5050
+Connection ~ 5100 4150
+Wire Wire Line
+	5100 5050 5100 5950
+Wire Wire Line
+	5100 5950 4750 5950
+Connection ~ 5100 5050
+Wire Wire Line
+	4900 5750 4900 6700
+Wire Wire Line
+	4900 6700 4750 6700
+Connection ~ 4900 5750
+Wire Wire Line
+	4900 6700 4900 7650
+Wire Wire Line
+	4900 7650 4750 7650
+Connection ~ 4900 6700
+Wire Wire Line
+	5000 5850 5000 6800
+Wire Wire Line
+	5000 6800 4750 6800
+Connection ~ 5000 5850
+Wire Wire Line
+	5000 6800 5000 7750
+Wire Wire Line
+	5000 7750 4750 7750
+Connection ~ 5000 6800
+Wire Wire Line
+	5100 5950 5100 6900
+Wire Wire Line
+	5100 6900 4750 6900
+Connection ~ 5100 5950
+Wire Wire Line
+	5100 6900 5100 7850
+Wire Wire Line
+	5100 7850 4750 7850
+Connection ~ 5100 6900
+$Comp
+L Device:Jumper_NC_Small JP1
+U 1 1 5BD89E80
+P 5550 1250
+F 0 "JP1" H 5550 1462 50  0000 C CNN
+F 1 "M0" H 5550 1371 50  0000 C CNN
+F 2 "Pin_Headers:Pin_Header_Straight_2x01_Pitch2.54mm" H 5550 1250 50  0001 C CNN
+F 3 "~" H 5550 1250 50  0001 C CNN
+	1    5550 1250
+	1    0    0    -1
+$EndComp
+$Comp
+L Device:Jumper_NC_Small JP2
+U 1 1 5BD89EC9
+P 5850 1350
+F 0 "JP2" H 5850 1562 50  0000 C CNN
+F 1 "M1" H 5850 1471 50  0000 C CNN
+F 2 "Pin_Headers:Pin_Header_Straight_2x01_Pitch2.54mm" H 5850 1350 50  0001 C CNN
+F 3 "~" H 5850 1350 50  0001 C CNN
+	1    5850 1350
+	1    0    0    -1
+$EndComp
+$Comp
+L Device:Jumper_NC_Small JP3
+U 1 1 5BD89F12
+P 6150 1450
+F 0 "JP3" H 6150 1662 50  0000 C CNN
+F 1 "M2" H 6150 1571 50  0000 C CNN
+F 2 "Pin_Headers:Pin_Header_Straight_2x01_Pitch2.54mm" H 6150 1450 50  0001 C CNN
+F 3 "~" H 6150 1450 50  0001 C CNN
+	1    6150 1450
+	1    0    0    -1
+$EndComp
+Wire Wire Line
+	4900 1250 5450 1250
+Connection ~ 4900 1250
+Wire Wire Line
+	5000 1350 5750 1350
+Connection ~ 5000 1350
+Wire Wire Line
+	5100 1450 6050 1450
+Connection ~ 5100 1450
+Wire Wire Line
+	6250 1450 6350 1450
+Wire Wire Line
+	6350 1450 6350 1350
+Wire Wire Line
+	6350 1350 5950 1350
+Wire Wire Line
+	6350 1350 6350 1250
+Wire Wire Line
+	6350 1250 5650 1250
+Connection ~ 6350 1350
+Wire Wire Line
+	6350 1250 6350 900
+Wire Wire Line
+	6350 900  3700 900
+Wire Wire Line
+	3700 900  3700 1550
+Connection ~ 6350 1250
+Connection ~ 3700 1550
+Text Label 5200 1250 0    50   ~ 0
+M0
+Text Label 5200 1350 0    50   ~ 0
+M1
+Text Label 5200 1450 0    50   ~ 0
+M2
 $EndSCHEMATC

Commit message: No real changes
Parts:
- CON1: symbol Connector:Conn_01x15_Female -> pump-rescue:Conn_01x15_Female-Connector
- JP1, JP2, JP3: symbol Device:Jumper_NC_Small -> pump-rescue:Jumper_NC_Small-Device
Changed lines of the file:
@@
 $EndSheet
 $Comp
-L Connector:Conn_01x15_Female CON1
+L pump-rescue:Conn_01x15_Female-Connector CON1
 U 1 1 5BCF8B18
 P 1750 4550
@@
 P7
 $Comp
-L power:PWR_FLAG #FLG0101
+L pump-rescue:PWR_FLAG-power #FLG0101
 U 1 1 5BD4DC20
 P 2900 3850
@@
 	2900 3850 3800 3850
 $Comp
-L power:PWR_FLAG #FLG0102
+L pump-rescue:PWR_FLAG-power #FLG0102
 U 1 1 5BD4DC4D
 P 3100 3950
@@
 Connection ~ 5100 6900
 $Comp
-L Device:Jumper_NC_Small JP1
+L pump-rescue:Jumper_NC_Small-Device JP1
 U 1 1 5BD89E80
 P 5550 1250
@@
 $EndComp
 $Comp
-L Device:Jumper_NC_Small JP2
+L pump-rescue:Jumper_NC_Small-Device JP2
 U 1 1 5BD89EC9
 P 5850 1350
@@
 $EndComp
 $Comp
-L Device:Jumper_NC_Small JP3
+L pump-rescue:Jumper_NC_Small-Device JP3
 U 1 1 5BD89F12
 P 6150 1450
